File: DeepSpace/DeepSpace.brd (EAGLE design)
At the start: 83.8 x 57.1 mm, 51 parts

Commit message: Verified Deep Space, Zeus
Parts:
- added R18: 1k, resistors:R0207/3
- A15, A16, A17: device potentiometers:16MM_PADS.3 -> potentiometers:16MM_B.MOUNT
- R17: value 560 -> 20k
- moved OUT 2.03 mm to (15.7, 3.81)
- moved GI 2.03 mm to (11.2, 3.81)
- moved GO 2.03 mm to (19.3, 3.81)
- moved ΙΝ 2.03 mm to (7.62, 3.81)
- moved STEPUP 1.02 mm to (30.1, 7.62)
- moved R6 0.76 mm to (41.4, 15.2)
Connections:
- net GND_15: now also R18.2
- net INR: now also R18.1
Routing:
- net N$2: track 19.0 -> 16.7 mm
- net INR: track 29.3 -> 31.3 mm
- net OUT: track 11.0 -> 8.96 mm
- net IN: track 30.5 -> 28.5 mm
- net -VC: track 27.3 -> 28.5 mm
- net N$20: track 14.8 -> 14.1 mm
