File: DeepSpace/DeepSpace.sch (EAGLE design)
At the start: 51 parts

Commit message: Verified Deep Space, Zeus
Parts:
- added R18: 1k, resistors:RESISTORS.3B
- A15, A16, A17: device potentiometers:16MM -> potentiometers:16MM.1
- R17: value 560 -> 20k
Connections:
- net GND_15: now also R18.2
- net INR: now also R18.1
