File: Randys_Gut/Randys_Gut.brd (EAGLE design)
At the start: 55.9 x 38.1 mm, 31 parts, among them Q1 2N1711, Q2 1N1711

Commit message: Minor Changes
Parts:
- C1: value (none) -> 47uF
- Q2: value 1N1711 -> 2N1711
Changed lines of the file:
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@@
 <attribute name="NAME" x="17.280459375" y="17.7861" size="1.016" layer="21" ratio="10" rot="R90" align="center"/>
 </element>
-<element name="Q2" library="transistors-BJT" package="TO18" value="1N1711" x="27.948459375" y="24.1361" smashed="yes" rot="R90">
+<element name="Q2" library="transistors-BJT" package="TO18" value="2N1711" x="27.948459375" y="24.1361" smashed="yes" rot="R90">
 <attribute name="NAME" x="26.170459375" y="24.1361" size="1.016" layer="21" ratio="10" rot="R90" align="center"/>
 </element>
@@
 <attribute name="NAME" x="36.87726875" y="23.565740625" size="1.016" layer="25" ratio="10" align="center"/>
 </element>
-<element name="C1" library="caps-elec" package="063_025" value="" x="19.03376875" y="25.407240625" smashed="yes">
+<element name="C1" library="caps-elec" package="063_025" value="47uF" x="19.03376875" y="25.407240625" smashed="yes">
 <attribute name="NAME" x="19.09726875" y="23.565740625" size="1.016" layer="25" ratio="10" align="center"/>
 <attribute name="VALUE" x="17.56376875" y="20.851240625" size="1.27" layer="27" ratio="12"/>

Commit message: Verified Deep Space, Zeus
Parts:
- BIAS, GREESE, LEVEL, TONE: device potentiometers:16MM_PADS.3 -> potentiometers:16MM_B.MOUNT
Changed lines of the file:
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@@
 <setting verticaltext="up"/>
 </settings>
-<grid distance="0.05" unitdist="inch" unit="inch" style="lines" multiple="1" display="yes" altdistance="0.001" altunitdist="inch" altunit="inch"/>
+<grid distance="0.01" unitdist="inch" unit="inch" style="lines" multiple="1" display="no" altdistance="0.001" altunitdist="inch" altunit="inch"/>
 <layers>
 <layer number="1" name="Top" color="4" fill="1" visible="yes" active="yes"/>
@@
 <layer number="25" name="tNames" color="7" fill="1" visible="yes" active="yes"/>
 <layer number="26" name="bNames" color="7" fill="1" visible="yes" active="yes"/>
-<layer number="27" name="tValues" color="7" fill="1" visible="yes" active="yes"/>
-<layer number="28" name="bValues" color="7" fill="1" visible="yes" active="yes"/>
+<layer number="27" name="tValues" color="7" fill="1" visible="no" active="yes"/>
+<layer number="28" name="bValues" color="7" fill="1" visible="no" active="yes"/>
 <layer number="29" name="tStop" color="7" fill="3" visible="no" active="yes"/>
 <layer number="30" name="bStop" color="7" fill="6" visible="no" active="yes"/>
@@
 <layer number="37" name="tTest" color="7" fill="1" visible="no" active="yes"/>
 <layer number="38" name="bTest" color="7" fill="1" visible="no" active="yes"/>
-<layer number="39" name="tKeepout" color="4" fill="11" visible="no" active="yes"/>
-<layer number="40" name="bKeepout" color="1" fill="11" visible="no" active="yes"/>
-<layer number="41" name="tRestrict" color="4" fill="10" visible="no" active="yes"/>
-<layer number="42" name="bRestrict" color="1" fill="10" visible="no" active="yes"/>
+<layer number="39" name="tKeepout" color="4" fill="11" visible="yes" active="yes"/>
+<layer number="40" name="bKeepout" color="1" fill="11" visible="yes" active="yes"/>
+<layer number="41" name="tRestrict" color="4" fill="10" visible="yes" active="yes"/>
+<layer number="42" name="bRestrict" color="1" fill="10" visible="yes" active="yes"/>
 <layer number="43" name="vRestrict" color="2" fill="10" visible="no" active="yes"/>
 <layer number="44" name="Drills" color="7" fill="1" visible="no" active="yes"/>
@@
 <layer number="49" name="Reference" color="7" fill="1" visible="no" active="yes"/>
 <layer number="50" name="dxf" color="7" fill="1" visible="no" active="no"/>
-<layer number="51" name="tDocu" color="7" fill="1" visible="no" active="yes"/>
-<layer number="52" name="bDocu" color="7" fill="1" visible="no" active="yes"/>
+<layer number="51" name="tDocu" color="7" fill="1" visible="yes" active="yes"/>
+<layer number="52" name="bDocu" color="7" fill="1" visible="yes" active="yes"/>
 <layer number="53" name="tGND_GNDA" color="7" fill="9" visible="no" active="no"/>
 <layer number="54" name="bGND_GNDA" color="1" fill="9" visible="no" active="no"/>
@@
 <layer number="107" name="BD-Top" color="7" fill="1" visible="no" active="yes"/>
 <layer number="151" name="HeatSink" color="7" fill="1" visible="no" active="yes"/>
-<layer number="200" name="200bmp" color="1" fill="10" visible="yes" active="yes"/>
+<layer number="200" name="200bmp" color="1" fill="10" visible="no" active="yes"/>
 <layer number="201" name="201bmp" color="7" fill="1" visible="no" active="yes"/>
 <layer number="250" name="Descript" color="7" fill="1" visible="no" active="yes"/>
@@
 <attribute name="NAME" x="27.948459375" y="35.8836" size="0.8128" layer="25" rot="R180" align="center"/>
 </element>
-<element name="BIAS" library="potentiometers" package="16MM_PADS.3" value="B5k" x="10.168459375" y="33.0261" smashed="yes">
+<element name="BIAS" library="potentiometers" package="16MM_B.MOUNT" value="B5k" x="10.168459375" y="33.0261" smashed="yes">
 <attribute name="NAME" x="10.168459375" y="35.6931" size="1.27" layer="26" ratio="10" rot="MR0" align="center"/>
 </element>
@@
 <attribute name="NAME" x="26.856259375" y="30.4861" size="1.016" layer="25" ratio="10" align="center-left"/>
 </element>
-<element name="GREESE" library="potentiometers" package="16MM_PADS.3" value="A100K" x="10.168459375" y="5.0861" smashed="yes">
+<element name="GREESE" library="potentiometers" package="16MM_B.MOUNT" value="A100K" x="10.168459375" y="5.0861" smashed="yes">
 <attribute name="NAME" x="10.168459375" y="2.6731" size="1.27" layer="26" ratio="10" rot="MR0" align="center"/>
 </element>
@@
 <attribute name="NAME" x="25.408459375" y="5.0861" size="0.8128" layer="25" ratio="10" align="bottom-center"/>
 </element>
-<element name="LEVEL" library="potentiometers" package="16MM_PADS.3" value="A100k" x="45.728459375" y="5.0861" smashed="yes">
+<element name="LEVEL" library="potentiometers" package="16MM_B.MOUNT" value="A100k" x="45.728459375" y="5.0861" smashed="yes">
 <attribute name="NAME" x="45.728459375" y="2.6731" size="1.27" layer="26" ratio="10" rot="MR0" align="center"/>
 </element>
@@
 <attribute name="NAME" x="45.728459375" y="27.46985" size="1.016" layer="25" font="vector" ratio="10" align="bottom-center"/>
 </element>
-<element name="TONE" library="potentiometers" package="16MM_PADS.3" value="B50k" x="45.728459375" y="33.0261" smashed="yes">
+<element name="TONE" library="potentiometers" package="16MM_B.MOUNT" value="B50k" x="45.728459375" y="33.0261" smashed="yes">
 <attribute name="NAME" x="45.728459375" y="35.4391" size="1.27" layer="26" ratio="10" rot="MR0" align="center"/>
 </element>
