File: Randys_Gut/Randys_Gut.brd (EAGLE design)
At the start: 55.9 x 38.1 mm, 31 parts, among them Q1 2N1711, Q2 2N1711

Commit message: Adding Photos
Parts:
- moved C6 2.55 mm to (37.1, 27.9)
- moved C1 2.30 mm to (19.3, 27.7)
- moved C3 1.48 mm to (29.2, 17.0)
- moved C4 1.48 mm to (29.2, 13.2)
- moved C5 1.48 mm to (29.2, 9.40)
- moved 4001 1.27 mm to (27.9, 31.8)
- moved C2 1.08 mm to (19.8, 9.40)
- moved PWR 1.02 mm to (27.9, 35.3)
- moved Q1 0.80 mm to (19.8, 18.0)
- moved Q2 0.51 mm to (27.9, 24.6)
Routing:
- net N$6: track 31.4 -> 34.7 mm
- net C3: track 21.6 -> 24.5 mm
- net N$8: track 49.5 -> 47.2 mm
- net N$5: track 26.1 -> 27.8 mm
- net N$7: track 27.5 -> 26.7 mm
