File: Randys_Gut/Randys_Gut.sch (EAGLE design)
At the start: 31 parts, among them Q1 2N1711, Q2 1N1711

Commit message: Minor Changes
Parts:
- C1: value (none) -> 47uF
- Q2: value 1N1711 -> 2N1711
Changed lines of the file:
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@@
 <part name="LEVEL" library="potentiometers" deviceset="16MM" device="" value="A100k"/>
 <part name="Q1" library="transistors-BJT" deviceset="2N2222A" device="" value="2N1711"/>
-<part name="Q2" library="transistors-BJT" deviceset="2N2222A" device="" value="1N1711"/>
+<part name="Q2" library="transistors-BJT" deviceset="2N2222A" device="" value="2N1711"/>
 <part name="C7" library="caps-elec" deviceset="050" device="1" value="22uF"/>
 <part name="GND2" library="supply pins" deviceset="GND" device=""/>
@@
 <part name="GO" library="supply pins" deviceset="GND_PAD" device="ROUND"/>
 <part name="C6" library="caps-elec" deviceset="063" device="1" value="100uF"/>
-<part name="C1" library="caps-elec" deviceset="063" device="1"/>
+<part name="C1" library="caps-elec" deviceset="063" device="1" value="47uF"/>
 </parts>
 <sheets>

Commit message: Verified Deep Space, Zeus
Parts:
- BIAS, GREESE, LEVEL, TONE: device potentiometers:16MM -> potentiometers:16MM.1
Changed lines of the file:
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@@
 <grid distance="0.1" unitdist="inch" unit="inch" style="lines" multiple="1" display="no" altdistance="0.01" altunitdist="inch" altunit="inch"/>
 <layers>
-<layer number="1" name="Top" color="4" fill="1" visible="no" active="no"/>
-<layer number="16" name="Bottom" color="1" fill="1" visible="no" active="no"/>
-<layer number="17" name="Pads" color="2" fill="1" visible="no" active="no"/>
-<layer number="18" name="Vias" color="2" fill="1" visible="no" active="no"/>
-<layer number="19" name="Unrouted" color="6" fill="1" visible="no" active="no"/>
-<layer number="20" name="Dimension" color="24" fill="1" visible="no" active="no"/>
-<layer number="21" name="tPlace" color="7" fill="1" visible="no" active="no"/>
-<layer number="22" name="bPlace" color="7" fill="1" visible="no" active="no"/>
-<layer number="23" name="tOrigins" color="15" fill="1" visible="no" active="no"/>
-<layer number="24" name="bOrigins" color="15" fill="1" visible="no" active="no"/>
-<layer number="25" name="tNames" color="7" fill="1" visible="no" active="no"/>
-<layer number="26" name="bNames" color="7" fill="1" visible="no" active="no"/>
-<layer number="27" name="tValues" color="7" fill="1" visible="no" active="no"/>
-<layer number="28" name="bValues" color="7" fill="1" visible="no" active="no"/>
+<layer number="1" name="Top" color="4" fill="1" visible="yes" active="no"/>
+<layer number="16" name="Bottom" color="1" fill="1" visible="yes" active="no"/>
+<layer number="17" name="Pads" color="2" fill="1" visible="yes" active="no"/>
+<layer number="18" name="Vias" color="2" fill="1" visible="yes" active="no"/>
+<layer number="19" name="Unrouted" color="6" fill="1" visible="yes" active="no"/>
+<layer number="20" name="Dimension" color="24" fill="1" visible="yes" active="no"/>
+<layer number="21" name="tPlace" color="7" fill="1" visible="yes" active="no"/>
+<layer number="22" name="bPlace" color="7" fill="1" visible="yes" active="no"/>
+<layer number="23" name="tOrigins" color="15" fill="1" visible="yes" active="no"/>
+<layer number="24" name="bOrigins" color="15" fill="1" visible="yes" active="no"/>
+<layer number="25" name="tNames" color="7" fill="1" visible="yes" active="no"/>
+<layer number="26" name="bNames" color="7" fill="1" visible="yes" active="no"/>
+<layer number="27" name="tValues" color="7" fill="1" visible="yes" active="no"/>
+<layer number="28" name="bValues" color="7" fill="1" visible="yes" active="no"/>
 <layer number="29" name="tStop" color="7" fill="3" visible="no" active="no"/>
 <layer number="30" name="bStop" color="7" fill="6" visible="no" active="no"/>
@@
 <layer number="35" name="tGlue" color="7" fill="4" visible="no" active="no"/>
 <layer number="36" name="bGlue" color="7" fill="5" visible="no" active="no"/>
-<layer number="37" name="tTest" color="7" fill="1" visible="no" active="no"/>
-<layer number="38" name="bTest" color="7" fill="1" visible="no" active="no"/>
+<layer number="37" name="tTest" color="7" fill="1" visible="yes" active="no"/>
+<layer number="38" name="bTest" color="7" fill="1" visible="yes" active="no"/>
 <layer number="39" name="tKeepout" color="4" fill="11" visible="no" active="no"/>
 <layer number="40" name="bKeepout" color="1" fill="11" visible="no" active="no"/>
@@
 <layer number="44" name="Drills" color="7" fill="1" visible="no" active="no"/>
 <layer number="45" name="Holes" color="7" fill="1" visible="no" active="no"/>
-<layer number="46" name="Milling" color="3" fill="1" visible="no" active="no"/>
-<layer number="47" name="Measures" color="7" fill="1" visible="no" active="no"/>
-<layer number="48" name="Document" color="7" fill="1" visible="no" active="no"/>
-<layer number="49" name="Reference" color="7" fill="1" visible="no" active="no"/>
-<layer number="50" name="dxf" color="7" fill="1" visible="no" active="no"/>
-<layer number="51" name="tDocu" color="7" fill="1" visible="no" active="no"/>
-<layer number="52" name="bDocu" color="7" fill="1" visible="no" active="no"/>
-<layer number="53" name="tGND_GNDA" color="7" fill="9" visible="no" active="no"/>
-<layer number="54" name="bGND_GNDA" color="1" fill="9" visible="no" active="no"/>
-<layer number="56" name="wert" color="7" fill="1" visible="no" active="no"/>
+<layer number="46" name="Milling" color="3" fill="1" visible="yes" active="no"/>
+<layer number="47" name="Measures" color="7" fill="1" visible="yes" active="no"/>
+<layer number="48" name="Document" color="7" fill="1" visible="yes" active="no"/>
+<layer number="49" name="Reference" color="7" fill="1" visible="yes" active="no"/>
+<layer number="50" name="dxf" color="7" fill="1" visible="yes" active="no"/>
+<layer number="51" name="tDocu" color="7" fill="1" visible="yes" active="no"/>
+<layer number="52" name="bDocu" color="7" fill="1" visible="yes" active="no"/>
+<layer number="53" name="tGND_GNDA" color="7" fill="9" visible="yes" active="no"/>
+<layer number="54" name="bGND_GNDA" color="1" fill="9" visible="yes" active="no"/>
+<layer number="56" name="wert" color="7" fill="1" visible="yes" active="no"/>
 <layer number="88" name="SimResults" color="9" fill="1" visible="yes" active="yes"/>
 <layer number="89" name="SimProbes" color="9" fill="1" visible="yes" active="yes"/>
@@
 <part name="4001" library="diodes" deviceset="DO41" device=".3" value="1N4001"/>
 <part name="PWR" library="jacks" deviceset="BATTERY" device="BAT2"/>
-<part name="GREESE" library="potentiometers" deviceset="16MM" device="" value="A100K"/>
-<part name="BIAS" library="potentiometers" deviceset="16MM" device="" value="B5k"/>
-<part name="TONE" library="potentiometers" deviceset="16MM" device="" value="B50k"/>
+<part name="GREESE" library="potentiometers" deviceset="16MM" device=".1" value="A100K"/>
+<part name="BIAS" library="potentiometers" deviceset="16MM" device=".1" value="B5k"/>
+<part name="TONE" library="potentiometers" deviceset="16MM" device=".1" value="B50k"/>
 <part name="R6" library="resistors_values" deviceset="RESISTORS" device=".3B" value="1M"/>
 <part name="R5" library="resistors" deviceset="RESISTORS" device=".3B" value="4.7k"/>
@@
 <part name="R8" library="resistors" deviceset="RESISTORS" device=".3B" value="22k"/>
 <part name="R7" library="resistors" deviceset="RESISTORS" device=".3B" value="68k"/>
-<part name="LEVEL" library="potentiometers" deviceset="16MM" device="" value="A100k"/>
+<part name="LEVEL" library="potentiometers" deviceset="16MM" device=".1" value="A100k"/>
 <part name="Q1" library="transistors-BJT" deviceset="2N2222A" device="" value="2N1711"/>
 <part name="Q2" library="transistors-BJT" deviceset="2N2222A" device="" value="2N1711"/>

Commit message: Adding Photos
Other:
- moved on the sheet: 4001, C10, C6, C7, C9, LEVEL, OUT, R7, R8, TONE
