File: Zeus/Zeus.brd (EAGLE design)
At the start: 61 x 38.9 mm, 27 parts, among them Q1 2N3903, Q2 2N3903, Q3 2N3903

Commit message: Minor Changes
Parts:
- FUZZ: value B25k -> B5k
Changed lines of the file:
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@@
 <attribute name="NAME" x="30.478553125" y="21.208265625" size="1.016" layer="25" ratio="10" rot="R180" align="center"/>
 </element>
-<element name="FUZZ" library="potentiometers" package="16MM_PADS.3" value="B25k" x="10.158553125" y="33.019265625" smashed="yes">
+<element name="FUZZ" library="potentiometers" package="16MM_PADS.3" value="B5k" x="10.158553125" y="33.019265625" smashed="yes">
 <attribute name="NAME" x="10.158553125" y="30.352265625" size="1.27" layer="26" ratio="10" rot="MR0" align="center"/>
 </element>

Commit message: Verified Deep Space, Zeus
Parts:
- FUZZ, LEVEL, TOP: device potentiometers:16MM_PADS.3 -> potentiometers:16MM_B.MOUNT
Changed lines of the file:
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@@
 <setting verticaltext="up"/>
 </settings>
-<grid distance="0.005" unitdist="inch" unit="inch" style="lines" multiple="1" display="yes" altdistance="0.001" altunitdist="inch" altunit="inch"/>
+<grid distance="0.01" unitdist="inch" unit="inch" style="lines" multiple="1" display="yes" altdistance="0.001" altunitdist="inch" altunit="inch"/>
 <layers>
 <layer number="1" name="Top" color="4" fill="1" visible="yes" active="yes"/>
@@
 <layer number="37" name="tTest" color="7" fill="1" visible="no" active="yes"/>
 <layer number="38" name="bTest" color="7" fill="1" visible="no" active="yes"/>
-<layer number="39" name="tKeepout" color="4" fill="11" visible="no" active="yes"/>
-<layer number="40" name="bKeepout" color="1" fill="11" visible="no" active="yes"/>
-<layer number="41" name="tRestrict" color="4" fill="10" visible="no" active="yes"/>
-<layer number="42" name="bRestrict" color="1" fill="10" visible="no" active="yes"/>
+<layer number="39" name="tKeepout" color="4" fill="11" visible="yes" active="yes"/>
+<layer number="40" name="bKeepout" color="1" fill="11" visible="yes" active="yes"/>
+<layer number="41" name="tRestrict" color="4" fill="10" visible="yes" active="yes"/>
+<layer number="42" name="bRestrict" color="1" fill="10" visible="yes" active="yes"/>
 <layer number="43" name="vRestrict" color="2" fill="10" visible="no" active="yes"/>
 <layer number="44" name="Drills" color="7" fill="1" visible="no" active="yes"/>
@@
 <layer number="49" name="Reference" color="7" fill="1" visible="no" active="yes"/>
 <layer number="50" name="dxf" color="7" fill="1" visible="no" active="no"/>
-<layer number="51" name="tDocu" color="7" fill="1" visible="no" active="yes"/>
-<layer number="52" name="bDocu" color="7" fill="1" visible="no" active="yes"/>
+<layer number="51" name="tDocu" color="7" fill="1" visible="yes" active="yes"/>
+<layer number="52" name="bDocu" color="7" fill="1" visible="yes" active="yes"/>
 <layer number="53" name="tGND_GNDA" color="7" fill="1" visible="no" active="no"/>
 <layer number="54" name="bGND_GNDA" color="7" fill="1" visible="no" active="no"/>
@@
 <attribute name="NAME" x="30.478553125" y="21.208265625" size="1.016" layer="25" ratio="10" rot="R180" align="center"/>
 </element>
-<element name="FUZZ" library="potentiometers" package="16MM_PADS.3" value="B5k" x="10.158553125" y="33.019265625" smashed="yes">
+<element name="FUZZ" library="potentiometers" package="16MM_B.MOUNT" value="B5k" x="10.158553125" y="33.019265625" smashed="yes">
 <attribute name="NAME" x="10.158553125" y="30.352265625" size="1.27" layer="26" ratio="10" rot="MR0" align="center"/>
 </element>
-<element name="TOP" library="potentiometers" package="16MM_PADS.3" value="B25k" x="30.478553125" y="10.159265625" smashed="yes">
+<element name="TOP" library="potentiometers" package="16MM_B.MOUNT" value="B25k" x="30.478553125" y="10.159265625" smashed="yes">
 <attribute name="NAME" x="30.478553125" y="12.572265625" size="1.27" layer="26" ratio="10" rot="MR0" align="center"/>
 </element>
-<element name="LEVEL" library="potentiometers" package="16MM_PADS.3" value="A100k" x="50.798553125" y="33.019265625" smashed="yes">
+<element name="LEVEL" library="potentiometers" package="16MM_B.MOUNT" value="A100k" x="50.798553125" y="33.019265625" smashed="yes">
 <attribute name="NAME" x="50.798553125" y="30.352265625" size="1.27" layer="26" ratio="10" rot="MR0" align="center"/>
 </element>
